Commit message: cleanup

File: urdf/.ipynb_checkpoints/akros_top.urdf-checkpoint.xacro (robot description, xacro)
@@ -1,8 +1,9 @@
 <?xml version="1.0"?>
 <robot name="akros_top" xmlns:xacro="http://ros.org/wiki/xacro">
-  <xacro:include filename="$(find depthai_ros_driver)/urdf/oakd.urdf.xacro"/>
   <xacro:include filename="$(find rplidar_ros)/urdf/rplidar.urdf.xacro"/>
+  <xacro:include filename="$(find depthai_bridge)/urdf/depthai_descr.urdf"/>
   <xacro:property name="M_PI"              value="3.1415926535897931" />
-  <xacro:property name="lidar_offset_yaw"  value="${3*M_PI/4}" />
+  <xacro:property name="lidar_offset_yaw"  value="${3*M_PI/4 - M_PI/12}" />
+  <xacro:property name="baseline"          value="0.075" />
   <xacro:arg name="oakd_offset_z"     default="0.100" />
   <xacro:arg name="oakd_offset_x"     default="0.038" />
@@ -16,5 +17,5 @@
     <origin xyz="$(arg oakd_offset_x) 0 $(arg oakd_offset_z)" rpy="0 0 0"/>
     <parent link="base_link"/>
-    <child link="depthai_base"/>
+    <child link="oakd_frame"/>
   </joint>
 </robot>

Commit message: separated rplidar stuff into single launch file

File: urdf/.ipynb_checkpoints/akros_top.urdf-checkpoint.xacro (robot description, xacro)
@@ -4,5 +4,5 @@
   <xacro:include filename="$(find depthai_bridge)/urdf/depthai_descr.urdf"/>
   <xacro:property name="M_PI"              value="3.1415926535897931" />
-  <xacro:property name="lidar_offset_yaw"  value="${3*M_PI/4 - M_PI/12}" />
+  <xacro:property name="lidar_offset_yaw"  value="${M_PI/2}" />
   <xacro:property name="baseline"          value="0.075" />
   <xacro:arg name="oakd_offset_z"     default="0.123" />

Commit message: updated launch files

File: urdf/.ipynb_checkpoints/akros_top.urdf-checkpoint.xacro (robot description, xacro)
@@ -7,14 +7,20 @@
   <xacro:property name="baseline"          value="0.075" />
   <xacro:arg name="oakd_offset_z"     default="0.123" />
-  <xacro:arg name="oakd_offset_x"     default="0.038" />
+  <xacro:arg name="oakd_offset_x"     default="-0.038" />
   <link name="base_link"/>
+  <link name="t265_link"/>
+  <joint name="t265_base_link" type="fixed">
+    <origin xyz="0 0 0" rpy="0 0 0"/>
+    <parent link="t265_link"/>
+    <child link="base_link"/>
+  </joint>
   <joint name="base2lidar_link" type="fixed">
-    <origin xyz="0 0 0" rpy="0 0 ${lidar_offset_yaw}"/>
-    <parent link="base_link"/>
+    <origin xyz="$(arg oakd_offset_x) 0 $(arg oakd_offset_z)" rpy="0 0 ${lidar_offset_yaw}"/>
+    <parent link="t265_link"/>
     <child link="rplidar_base"/>
   </joint>
   <joint name="base2oakd_link" type="fixed">
-    <origin xyz="$(arg oakd_offset_x) 0 $(arg oakd_offset_z)" rpy="0 0 0"/>
-    <parent link="base_link"/>
+    <origin xyz="0 0 0" rpy="0 0 0"/>
+    <parent link="t265_link"/>
     <child link="oakd_frame"/>
   </joint>

Commit message: added twist mux

File: urdf/.ipynb_checkpoints/akros_top.urdf-checkpoint.xacro (robot description, xacro)
@@ -9,18 +9,18 @@
   <xacro:arg name="oakd_offset_x"     default="-0.038" />
   <link name="base_link"/>
-  <link name="t265_link"/>
+  <link name="t265_pose_frame"/>
   <joint name="t265_base_link" type="fixed">
     <origin xyz="0 0 0" rpy="0 0 0"/>
-    <parent link="t265_link"/>
+    <parent link="t265_pose_frame"/>
     <child link="base_link"/>
   </joint>
   <joint name="base2lidar_link" type="fixed">
     <origin xyz="$(arg oakd_offset_x) 0 $(arg oakd_offset_z)" rpy="0 0 ${lidar_offset_yaw}"/>
-    <parent link="t265_link"/>
+    <parent link="base_link"/>
     <child link="rplidar_base"/>
   </joint>
   <joint name="base2oakd_link" type="fixed">
     <origin xyz="0 0 0" rpy="0 0 0"/>
-    <parent link="t265_link"/>
+    <parent link="base_link"/>
     <child link="oakd_frame"/>
   </joint>
