Commit message: updated bringup + slam with oakd

File: akros_description/urdf/akros_top.urdf.xacro (robot description, xacro)
@@ -5,7 +5,6 @@
   <xacro:property name="M_PI"              value="3.1415926535897931" />
   <xacro:property name="lidar_offset_yaw"  value="${M_PI/2}" />
-  <xacro:property name="baseline"          value="0.075" />
-  <xacro:arg name="oakd_offset_z"     default="0.123" />
-  <xacro:arg name="oakd_offset_x"     default="-0.038" />
+  <xacro:arg name="lidar_offset_z"     default="0.123" />
+  <xacro:arg name="lidar_offset_x"     default="-0.038" />
   <link name="base_link"/>
   <link name="t265_pose_frame"/>
@@ -16,5 +15,5 @@
   </joint>
   <joint name="base2lidar_link" type="fixed">
-    <origin xyz="$(arg oakd_offset_x) 0 $(arg oakd_offset_z)" rpy="0 0 ${lidar_offset_yaw}"/>
+    <origin xyz="$(arg lidar_offset_x) 0 $(arg lidar_offset_z)" rpy="0 0 ${lidar_offset_yaw}"/>
     <parent link="base_link"/>
     <child link="rplidar_base"/>
