Commit message: update

File: akros_description/urdf/akros.urdf.xacro (robot description, xacro)
@@ -1,14 +1,11 @@
 <?xml version="1.0"?>
 <robot name="akros_top" xmlns:xacro="http://ros.org/wiki/xacro">
-  <!-- xacro:include filename="$(find rplidar_ros)/urdf/rplidar.urdf.xacro"/ -->
-  <xacro:include filename="$(find depthai_bridge)/urdf/depthai_descr.urdf.xacro"/>
-  <xacro:property name="M_PI"              value="3.1415926535897931" />
-  <xacro:property name="rplidar_offset_yaw"  value="${M_PI/2}" />
+  <xacro:property name="M_PI"          value="3.1415926535897931" />
   <xacro:arg name="lidar_offset_z"     default="0.08" />
   <xacro:arg name="lidar_offset_x"     default="-0.08" />
+  <link name="t265_pose_frame"/>
   <link name="base_link"/>
   <link name="t265_link"/>
   <link name="laser_frame"/>
-  <link name="t265_pose_frame"/>
   <joint name="base_link_t265_dummy" type="fixed">
     <origin xyz="0 0 0" rpy="0 0 0"/>
@@ -26,8 +23,3 @@
     <child link="laser_frame"/>
   </joint>
-  <joint name="base_oakd_link" type="fixed">
-    <origin xyz="0 0 0" rpy="0 0 0"/>
-    <parent link="base_link"/>
-    <child link="oakd_link"/>
-  </joint>
 </robot>

Commit message: Update akros.urdf.xacro

File: akros_description/urdf/akros.urdf.xacro (robot description, xacro)
@@ -7,5 +7,5 @@
     <origin xyz="0 0 0" rpy="0 0 0" />
     <geometry>
-      <mesh filename="package://mecanum_car/meshes/navigation_module_centered.stl" />
+      <mesh filename="package://akros_description/meshes/navigation_module_centered.stl" />
     </geometry>
     <material name="">
@@ -38,14 +38,14 @@
     <origin xyz="0 0 0" rpy="0 0 0" />
     <geometry>
-      <mesh filename="package://mecanum_car/meshes/ld06.stl" />
-    </geometry>
-    <material name="">
-      <color rgba="0 0 0 1" />
-    </material>
-  </visual>
-  <collision>
-    <origin xyz="0 0 0" rpy="0 0 0" />
-    <geometry>
-      <mesh filename="package://mecanum_car/meshes/ld06.stl" />
+      <mesh filename="package://akros_description/meshes/ld06.stl" />
+    </geometry>
+    <material name="">
+      <color rgba="0 0 0 1" />
+    </material>
+  </visual>
+  <collision>
+    <origin xyz="0 0 0" rpy="0 0 0" />
+    <geometry>
+      <mesh filename="package://akros_description/meshes/ld06.stl" />
     </geometry>
   </collision>
@@ -63,5 +63,5 @@
     <origin xyz="0 0 0" rpy="0 0 0" />
     <geometry>
-      <mesh filename="package://mecanum_car/meshes/t265.stl" />
+      <mesh filename="package://akros_description/meshes/t265.stl" />
     </geometry>
     <material name="">
@@ -85,5 +85,5 @@
     <origin xyz="0 0 0" rpy="0 0 0" />
     <geometry>
-      <mesh filename="package://mecanum_car/meshes/base_module_centered.stl" />
+      <mesh filename="package://akros_description/meshes/base_module_centered.stl" />
     </geometry>
     <material name="">
@@ -107,5 +107,5 @@
     <origin xyz="0 0 0" rpy="0 0 0" />
     <geometry>
-      <mesh filename="package://mecanum_car/meshes/wheel_left_front.stl" />
+      <mesh filename="package://akros_description/meshes/wheel_left_front.stl" />
     </geometry>
     <material name="">
@@ -129,5 +129,5 @@
     <origin xyz="0 0 0" rpy="0 0 0" />
     <geometry>
-      <mesh filename="package://mecanum_car/meshes/wheel_left_back.stl" />
+      <mesh filename="package://akros_description/meshes/wheel_left_back.stl" />
     </geometry>
     <material name="">
@@ -151,5 +151,5 @@
     <origin xyz="0 0 0" rpy="0 0 0" />
     <geometry>
-      <mesh filename="package://mecanum_car/meshes/wheel_right_front.stl" />
+      <mesh filename="package://akros_description/meshes/wheel_right_front.stl" />
     </geometry>
     <material name="">
@@ -173,5 +173,5 @@
     <origin xyz="0 0 0" rpy="0 0 0" />
     <geometry>
-      <mesh filename="package://mecanum_car/meshes/wheel_right_back.stl" />
+      <mesh filename="package://akros_description/meshes/wheel_right_back.stl" />
     </geometry>
     <material name="">
