Commit message: Update akros_t265_only.urdf.xacro

File: akros_description/urdf/akros_t265_only.urdf.xacro (robot description, xacro)
@@ -7,5 +7,5 @@
     <origin xyz="0 0 0" rpy="0 0 0" />
     <geometry>
-      <mesh filename="package://mecanum_car/meshes/navigation_module_centered.stl" />
+      <mesh filename="package://akros_description/meshes/navigation_module_centered.stl" />
     </geometry>
     <material name="">
@@ -38,14 +38,14 @@
     <origin xyz="0 0 0" rpy="0 0 0" />
     <geometry>
-      <mesh filename="package://mecanum_car/meshes/ld06.stl" />
-    </geometry>
-    <material name="">
-      <color rgba="0 0 0 1" />
-    </material>
-  </visual>
-  <collision>
-    <origin xyz="0 0 0" rpy="0 0 0" />
-    <geometry>
-      <mesh filename="package://mecanum_car/meshes/ld06.stl" />
+      <mesh filename="package://akros_description/meshes/ld06.stl" />
+    </geometry>
+    <material name="">
+      <color rgba="0 0 0 1" />
+    </material>
+  </visual>
+  <collision>
+    <origin xyz="0 0 0" rpy="0 0 0" />
+    <geometry>
+      <mesh filename="package://akros_description/meshes/ld06.stl" />
     </geometry>
   </collision>
@@ -63,5 +63,5 @@
     <origin xyz="0 0 0" rpy="0 0 0" />
     <geometry>
-      <mesh filename="package://mecanum_car/meshes/t265.stl" />
+      <mesh filename="package://akros_description/meshes/t265.stl" />
     </geometry>
     <material name="">
@@ -87,5 +87,5 @@
     <origin xyz="0 0 0" rpy="0 0 0" />
     <geometry>
-      <mesh filename="package://mecanum_car/meshes/base_module_centered.stl" />
+      <mesh filename="package://akros_description/meshes/base_module_centered.stl" />
     </geometry>
     <material name="">
@@ -109,5 +109,5 @@
     <origin xyz="0 0 0" rpy="0 0 0" />
     <geometry>
-      <mesh filename="package://mecanum_car/meshes/wheel_left_front.stl" />
+      <mesh filename="package://akros_description/meshes/wheel_left_front.stl" />
     </geometry>
     <material name="">
@@ -131,5 +131,5 @@
     <origin xyz="0 0 0" rpy="0 0 0" />
     <geometry>
-      <mesh filename="package://mecanum_car/meshes/wheel_left_back.stl" />
+      <mesh filename="package://akros_description/meshes/wheel_left_back.stl" />
     </geometry>
     <material name="">
@@ -153,5 +153,5 @@
     <origin xyz="0 0 0" rpy="0 0 0" />
     <geometry>
-      <mesh filename="package://mecanum_car/meshes/wheel_right_front.stl" />
+      <mesh filename="package://akros_description/meshes/wheel_right_front.stl" />
     </geometry>
     <material name="">
@@ -175,5 +175,5 @@
     <origin xyz="0 0 0" rpy="0 0 0" />
     <geometry>
-      <mesh filename="package://mecanum_car/meshes/wheel_right_back.stl" />
+      <mesh filename="package://akros_description/meshes/wheel_right_back.stl" />
     </geometry>
     <material name="">
