Commit message: updated slam launch file

File: akros_description/urdf/.ipynb_checkpoints/akros_top.urdf-checkpoint.xacro (robot description, xacro)
@@ -2,5 +2,5 @@
 <robot name="akros_top" xmlns:xacro="http://ros.org/wiki/xacro">
   <xacro:include filename="$(find rplidar_ros)/urdf/rplidar.urdf.xacro"/>
-  <xacro:include filename="$(find depthai_bridge)/urdf/depthai_descr.urdf"/>
+  <xacro:include filename="$(find depthai_bridge)/urdf/depthai_descr.urdf.xacro"/>
   <xacro:property name="M_PI"              value="3.1415926535897931" />
   <xacro:property name="lidar_offset_yaw"  value="${M_PI/2}" />
@@ -23,5 +23,5 @@
     <origin xyz="0 0 0" rpy="0 0 0"/>
     <parent link="base_link"/>
-    <child link="oakd_frame"/>
+    <child link="oakd_link"/>
   </joint>
 </robot>

Commit message: added akros_teleop

File: akros_description/urdf/.ipynb_checkpoints/akros_top.urdf-checkpoint.xacro (robot description, xacro)
@@ -5,20 +5,25 @@
   <xacro:property name="M_PI"              value="3.1415926535897931" />
   <xacro:property name="lidar_offset_yaw"  value="${M_PI/2}" />
-  <xacro:property name="baseline"          value="0.075" />
-  <xacro:arg name="oakd_offset_z"     default="0.123" />
-  <xacro:arg name="oakd_offset_x"     default="-0.038" />
+  <xacro:arg name="lidar_offset_z"     default="0.12" />
+  <xacro:arg name="lidar_offset_x"     default="-0.1" />
   <link name="base_link"/>
+  <link name="t265_link"/>
   <link name="t265_pose_frame"/>
-  <joint name="t265_base_link" type="fixed">
+  <joint name="base_link_pose_dummy" type="fixed">
     <origin xyz="0 0 0" rpy="0 0 0"/>
     <parent link="t265_pose_frame"/>
     <child link="base_link"/>
   </joint>
-  <joint name="base2lidar_link" type="fixed">
-    <origin xyz="$(arg oakd_offset_x) 0 $(arg oakd_offset_z)" rpy="0 0 ${lidar_offset_yaw}"/>
+  <joint name="base_link_t265" type="fixed">
+    <origin xyz="0 0 0" rpy="0 0 0"/>
+    <parent link="base_link"/>
+    <child link="t265_link"/>
+  </joint>
+  <joint name="base_lidar_link" type="fixed">
+    <origin xyz="$(arg lidar_offset_x) 0 $(arg lidar_offset_z)" rpy="0 0 ${lidar_offset_yaw}"/>
     <parent link="base_link"/>
     <child link="rplidar_base"/>
   </joint>
-  <joint name="base2oakd_link" type="fixed">
+  <joint name="base_oakd_link" type="fixed">
     <origin xyz="0 0 0" rpy="0 0 0"/>
     <parent link="base_link"/>

File: akros_description/urdf/akros_top.urdf.xacro (robot description, xacro)
@@ -5,19 +5,25 @@
   <xacro:property name="M_PI"              value="3.1415926535897931" />
   <xacro:property name="lidar_offset_yaw"  value="${M_PI/2}" />
-  <xacro:arg name="lidar_offset_z"     default="0.123" />
-  <xacro:arg name="lidar_offset_x"     default="-0.038" />
+  <xacro:arg name="lidar_offset_z"     default="0.12" />
+  <xacro:arg name="lidar_offset_x"     default="-0.1" />
   <link name="base_link"/>
+  <link name="t265_link"/>
   <link name="t265_pose_frame"/>
-  <joint name="t265_base_link" type="fixed">
+  <joint name="base_link_pose_dummy" type="fixed">
     <origin xyz="0 0 0" rpy="0 0 0"/>
     <parent link="t265_pose_frame"/>
     <child link="base_link"/>
   </joint>
-  <joint name="base2lidar_link" type="fixed">
+  <joint name="base_link_t265" type="fixed">
+    <origin xyz="0 0 0" rpy="0 0 0"/>
+    <parent link="base_link"/>
+    <child link="t265_link"/>
+  </joint>
+  <joint name="base_lidar_link" type="fixed">
     <origin xyz="$(arg lidar_offset_x) 0 $(arg lidar_offset_z)" rpy="0 0 ${lidar_offset_yaw}"/>
     <parent link="base_link"/>
     <child link="rplidar_base"/>
   </joint>
-  <joint name="base2oakd_link" type="fixed">
+  <joint name="base_oakd_link" type="fixed">
     <origin xyz="0 0 0" rpy="0 0 0"/>
     <parent link="base_link"/>

Commit message: tune move_base

File: akros_description/urdf/.ipynb_checkpoints/akros_top.urdf-checkpoint.xacro (robot description, xacro)
@@ -1,12 +1,13 @@
 <?xml version="1.0"?>
 <robot name="akros_top" xmlns:xacro="http://ros.org/wiki/xacro">
-  <xacro:include filename="$(find rplidar_ros)/urdf/rplidar.urdf.xacro"/>
+  <!-- xacro:include filename="$(find rplidar_ros)/urdf/rplidar.urdf.xacro"/ -->
   <xacro:include filename="$(find depthai_bridge)/urdf/depthai_descr.urdf.xacro"/>
   <xacro:property name="M_PI"              value="3.1415926535897931" />
-  <xacro:property name="lidar_offset_yaw"  value="${M_PI/2}" />
-  <xacro:arg name="lidar_offset_z"     default="0.12" />
-  <xacro:arg name="lidar_offset_x"     default="-0.1" />
+  <xacro:property name="rplidar_offset_yaw"  value="${M_PI/2}" />
+  <xacro:arg name="lidar_offset_z"     default="0.08" />
+  <xacro:arg name="lidar_offset_x"     default="-0.08" />
   <link name="base_link"/>
   <link name="t265_link"/>
+  <link name="laser_frame"/>
   <link name="t265_pose_frame"/>
   <joint name="base_link_pose_dummy" type="fixed">
@@ -21,7 +22,7 @@
   </joint>
   <joint name="base_lidar_link" type="fixed">
-    <origin xyz="$(arg lidar_offset_x) 0 $(arg lidar_offset_z)" rpy="0 0 ${lidar_offset_yaw}"/>
+    <origin xyz="$(arg lidar_offset_x) 0 $(arg lidar_offset_z)" rpy="0 0 0"/>
     <parent link="base_link"/>
-    <child link="rplidar_base"/>
+    <child link="laser_frame"/>
   </joint>
   <joint name="base_oakd_link" type="fixed">

Commit message: added frontier_exploration, and assisted_teleop to auto mode

File: akros_description/urdf/.ipynb_checkpoints/akros_top.urdf-checkpoint.xacro (robot description, xacro)
@@ -2,9 +2,10 @@
 <robot name="akros_top" xmlns:xacro="http://ros.org/wiki/xacro">
   <!-- xacro:include filename="$(find rplidar_ros)/urdf/rplidar.urdf.xacro"/ -->
-  <xacro:include filename="$(find depthai_bridge)/urdf/depthai_descr.urdf.xacro"/>
+  <!-- xacro:include filename="$(find depthai_bridge)/urdf/depthai_descr.urdf.xacro"/ -->
   <xacro:property name="M_PI"              value="3.1415926535897931" />
   <xacro:property name="rplidar_offset_yaw"  value="${M_PI/2}" />
   <xacro:arg name="lidar_offset_z"     default="0.08" />
   <xacro:arg name="lidar_offset_x"     default="-0.08" />
+  <link name="oakd_link"/>
   <link name="base_link"/>
   <link name="t265_link"/>

Commit message: added rgbd inertial node and nodelet

File: akros_description/urdf/.ipynb_checkpoints/akros_top.urdf-checkpoint.xacro (robot description, xacro)
@@ -2,10 +2,10 @@
 <robot name="akros_top" xmlns:xacro="http://ros.org/wiki/xacro">
   <!-- xacro:include filename="$(find rplidar_ros)/urdf/rplidar.urdf.xacro"/ -->
-  <!-- xacro:include filename="$(find depthai_bridge)/urdf/depthai_descr.urdf.xacro"/ -->
+  <xacro:include filename="$(find depthai_bridge)/urdf/depthai_descr.urdf.xacro"/>
   <xacro:property name="M_PI"              value="3.1415926535897931" />
   <xacro:property name="rplidar_offset_yaw"  value="${M_PI/2}" />
   <xacro:arg name="lidar_offset_z"     default="0.08" />
   <xacro:arg name="lidar_offset_x"     default="-0.08" />
-  <link name="oakd_link"/>
+  <!-- link name="oakd_link"/ -->
   <link name="base_link"/>
   <link name="t265_link"/>

Commit message: updated wheel odometry, removed assisted teleop, mode subscriber on Arduino

File: akros_description/urdf/.ipynb_checkpoints/akros_top.urdf-checkpoint.xacro (robot description, xacro)
@@ -1,5 +1,4 @@
 <?xml version="1.0"?>
 <robot name="akros_top" xmlns:xacro="http://ros.org/wiki/xacro">
-  <!-- xacro:include filename="$(find rplidar_ros)/urdf/rplidar.urdf.xacro"/ -->
   <xacro:include filename="$(find depthai_bridge)/urdf/depthai_descr.urdf.xacro"/>
   <xacro:property name="M_PI"              value="3.1415926535897931" />
@@ -7,18 +6,11 @@
   <xacro:arg name="lidar_offset_z"     default="0.08" />
   <xacro:arg name="lidar_offset_x"     default="-0.08" />
-  <!-- link name="oakd_link"/ -->
   <link name="base_link"/>
-  <link name="t265_link"/>
   <link name="laser_frame"/>
-  <link name="t265_pose_frame"/>
-  <joint name="base_link_pose_dummy" type="fixed">
+  <link name="enc_pose_frame"/>
+  <joint name="base_link_enc_dummy" type="fixed">
     <origin xyz="0 0 0" rpy="0 0 0"/>
-    <parent link="t265_pose_frame"/>
+    <parent link="enc_pose_frame"/>
     <child link="base_link"/>
-  </joint>
-  <joint name="base_link_t265" type="fixed">
-    <origin xyz="0 0 0" rpy="0 0 0"/>
-    <parent link="base_link"/>
-    <child link="t265_link"/>
   </joint>
   <joint name="base_lidar_link" type="fixed">

File: akros_description/urdf/akros_top_t265.urdf.xacro (robot description, xacro)
@@ -1,4 +1,5 @@
 <?xml version="1.0"?>
 <robot name="akros_top" xmlns:xacro="http://ros.org/wiki/xacro">
+  <!-- xacro:include filename="$(find rplidar_ros)/urdf/rplidar.urdf.xacro"/ -->
   <xacro:include filename="$(find depthai_bridge)/urdf/depthai_descr.urdf.xacro"/>
   <xacro:property name="M_PI"              value="3.1415926535897931" />
@@ -7,10 +8,16 @@
   <xacro:arg name="lidar_offset_x"     default="-0.08" />
   <link name="base_link"/>
+  <link name="t265_link"/>
   <link name="laser_frame"/>
-  <link name="enc_pose_frame"/>
-  <joint name="base_link_enc_dummy" type="fixed">
+  <link name="t265_pose_frame"/>
+  <joint name="base_link_t265_dummy" type="fixed">
     <origin xyz="0 0 0" rpy="0 0 0"/>
-    <parent link="enc_pose_frame"/>
+    <parent link="t265_pose_frame"/>
     <child link="base_link"/>
+  </joint>
+  <joint name="base_link_t265" type="fixed">
+    <origin xyz="0 0 0" rpy="0 0 0"/>
+    <parent link="base_link"/>
+    <child link="t265_link"/>
   </joint>
   <joint name="base_lidar_link" type="fixed">
