Commit message: update urdf

File: akros_description/urdf/.ipynb_checkpoints/akros_t265_only.urdf-checkpoint.xacro (robot description, xacro)
@@ -1,7 +1,9 @@
 <?xml version="1.0"?>
 <robot name="akros_top" xmlns:xacro="http://ros.org/wiki/xacro">
-  <xacro:property name="M_PI"          value="3.1415926535897931" />
-  <xacro:arg name="lidar_offset_z"     default="0.08" />
-  <xacro:arg name="lidar_offset_x"     default="-0.08" />
+  <xacro:property name="M_PI"         value="3.1415926535897931" />
+  <xacro:arg name="lidar_offset_z"    default="0.07" />
+  <xacro:arg name="lidar_offset_x"    default="-0.08" />
+  <xacro:arg name="t265_offset_z"     default="0.01225" />
+  <xacro:arg name="t265_offset_x"     default="0.1" />
   <link name="t265_pose_frame"/>
   <link name="base_link"/>
@@ -9,15 +11,15 @@
   <link name="laser_frame"/>
   <joint name="base_link_t265_dummy" type="fixed">
-    <origin xyz="0 0 0" rpy="0 0 0"/>
+    <origin xyz="-$(arg t265_offset_x) 0 -$(arg t265_offset_z)" rpy="0 0 0"/>
     <parent link="t265_pose_frame"/>
     <child link="base_link"/>
   </joint>
   <joint name="base_link_t265" type="fixed">
-    <origin xyz="0 0 0" rpy="0 0 0"/>
+    <origin xyz="$(arg t265_offset_x) 0 $(arg t265_offset_z)" rpy="0 0 0"/>
     <parent link="base_link"/>
     <child link="t265_link"/>
   </joint>
   <joint name="base_lidar_link" type="fixed">
-    <origin xyz="$(arg lidar_offset_x) 0 $(arg lidar_offset_z)" rpy="0 0 0"/>
+    <origin xyz="0 0 $(arg lidar_offset_z)" rpy="0 0 0"/>
     <parent link="base_link"/>
     <child link="laser_frame"/>

File: akros_description/urdf/.ipynb_checkpoints/akros_t265_with_encoders.urdf-checkpoint.xacro (robot description, xacro)
@@ -1,17 +1,18 @@
 <?xml version="1.0"?>
 <robot name="akros_top" xmlns:xacro="http://ros.org/wiki/xacro">
-  <xacro:property name="M_PI"          value="3.1415926535897931" />
-  <xacro:arg name="lidar_offset_z"     default="0.08" />
-  <xacro:arg name="lidar_offset_x"     default="-0.08" />
+  <xacro:property name="M_PI"         value="3.1415926535897931" />
+  <xacro:arg name="lidar_offset_z"    default="0.07" />
+  <xacro:arg name="t265_offset_z"     default="0.01225" />
+  <xacro:arg name="t265_offset_x"     default="0.1" />
   <link name="t265_pose_frame"/>
   <link name="base_link"/>
   <link name="laser_frame"/>
   <joint name="base_link_t265" type="fixed">
-    <origin xyz="0 0 0" rpy="0 0 0"/>
+    <origin xyz="$(arg t265_offset_x) 0 $(arg t265_offset_z)" rpy="0 0 0"/>
     <parent link="base_link"/>
     <child link="t265_pose_frame"/>
   </joint>
   <joint name="base_lidar_link" type="fixed">
-    <origin xyz="$(arg lidar_offset_x) 0 $(arg lidar_offset_z)" rpy="0 0 0"/>
+    <origin xyz="0 0 $(arg lidar_offset_z)" rpy="0 0 0"/>
     <parent link="base_link"/>
     <child link="laser_frame"/>
