Commit message: update urdf and meshes

File: akros_description/urdf/.ipynb_checkpoints/akros.urdf-checkpoint.xacro (robot description, xacro)
@@ -4,4 +4,22 @@
 <!-- NAVIGATION MODULE (BASE_LINK) -->
 <link name="base_link">
+  <visual>
+    <origin xyz="0 0 0" rpy="0 0 0" />
+    <geometry>
+      <mesh filename="package://mecanum_car/meshes/navigation_module_centered.stl" />
+    </geometry>
+    <material name="">
+      <color rgba="1 1 1 1" />
+    </material>
+  </visual>
+  <collision>
+    <origin xyz="0 0 0" rpy="0 0 0" />
+    <geometry>
+      <box size='0.21 0.15 0.02'/>
+    </geometry>
+  </collision>
+</link>
+<!-- BASE_LINK_INERTIAL (WORKAROUND FOR KDL) -->
+<link name="base_link_inertial">
   <inertial>
     <origin xyz="0 0 0" rpy="0 0 0" />
@@ -9,19 +27,4 @@
     <inertia ixx="0.01" ixy="0.01" ixz="0.01" iyy="0.01" iyz="0.01" izz="0.01" />
   </inertial>
-  <visual>
-    <origin xyz="0 0 0" rpy="0 0 0" />
-    <geometry>
-      <mesh filename="package://mecanum_car/meshes/navigation_module_rsz.stl" />
-    </geometry>
-    <material name="">
-      <color rgba="1 1 1 1" />
-    </material>
-  </visual>
-  <collision>
-    <origin xyz="0 0 0" rpy="0 0 0" />
-    <geometry>
-      <box size='0.21 0.15 0.02'/>
-    </geometry>
-  </collision>
 </link>
 <!-- LD06 LIDAR -->
@@ -182,4 +185,10 @@
 </link>
 <!-- **** JOINTS **** -->
+<!-- BASE_LINK_INERTIAL TO BASE_LINK -->
+<joint name="base_inertial_fixed" type="fixed">
+  <parent link="base_link"/>
+  <child link="base_link_inertial"/>
+  <origin xyz="0 0 0"/>
+</joint>
 <!-- LASER_FRAME TO BASE_LINK -->
 <joint name="base_lidar_fixed" type="fixed">

Commit message: add glb files and updated mesh_pub

File: akros_description/urdf/.ipynb_checkpoints/akros.urdf-checkpoint.xacro (robot description, xacro)
@@ -20,5 +20,5 @@
   </collision>
 </link>
-<!-- BASE_LINK_INERTIAL (WORKAROUND FOR KDL) -->
+<!-- BASE_LINK_INERTIAL (WORKAROUND FOR KDL WHICH DOES NOT ACCEPT BASE_LINK WITH INERTIA) -->
 <link name="base_link_inertial">
   <inertial>
@@ -28,6 +28,6 @@
   </inertial>
 </link>
-<!-- LD06 LIDAR -->
-<link name="laser_frame">
+<!-- LD06 LASER_LINK -->
+<link name="laser_link">
   <inertial>
     <origin xyz="0 0 0" rpy="0 0 0" />
@@ -51,5 +51,7 @@
   </collision>
 </link>
-<!-- T265 TRACKING CAMERA -->
+<!-- LASER_FRAME -->
+<link name="laser_frame"/>
+<!-- T265 TRACKING CAMERA (T265_POSE_FRAME AS WORKAROUND TO KEEP TREE CONTINUOUS)-->
 <link name="t265_pose_frame">
   <inertial>
@@ -191,9 +193,15 @@
   <origin xyz="0 0 0"/>
 </joint>
-<!-- LASER_FRAME TO BASE_LINK -->
+<!-- LASER_LINK TO BASE_LINK -->
 <joint name="base_lidar_fixed" type="fixed">
   <parent link="base_link"/>
+  <child link="laser_link"/>
+  <origin xyz="0 0 0.0415"/>
+</joint>
+<!-- LASER_FRAME TO LASER_LINK -->
+<joint name="laser_frame_fixed" type="fixed">
+  <parent link="laser_link"/>
   <child link="laser_frame"/>
-  <origin xyz="0 0 0.0415"/>
+  <origin xyz="0 0 0.03"/>
 </joint>
 <!-- T265_POSE_FRAME TO BASE_LINK -->
@@ -205,5 +213,5 @@
 <!-- BASE_FOOTPRINT TO BASE_LINK -->
 <joint name="base_link_footprint_fixed" type="fixed">
-  <origin xyz="0 0 -0.063" rpy="0 0 0"/>
+  <origin xyz="0 0 -0.099" rpy="0 0 0"/>
   <parent link="base_link"/>
   <child link="base_footprint"/>

File: akros_description/urdf/akros.urdf.xacro (robot description, xacro)
@@ -20,5 +20,5 @@
   </collision>
 </link>
-<!-- BASE_LINK_INERTIAL (WORKAROUND FOR KDL) -->
+<!-- BASE_LINK_INERTIAL (WORKAROUND FOR KDL WHICH DOES NOT ACCEPT BASE_LINK WITH INERTIA) -->
 <link name="base_link_inertial">
   <inertial>
@@ -28,6 +28,6 @@
   </inertial>
 </link>
-<!-- LD06 LIDAR -->
-<link name="laser_frame">
+<!-- LD06 LASER_LINK -->
+<link name="laser_link">
   <inertial>
     <origin xyz="0 0 0" rpy="0 0 0" />
@@ -51,5 +51,7 @@
   </collision>
 </link>
-<!-- T265 TRACKING CAMERA -->
+<!-- LASER_FRAME -->
+<link name="laser_frame"/>
+<!-- T265 TRACKING CAMERA (T265_POSE_FRAME AS WORKAROUND TO KEEP TREE CONTINUOUS)-->
 <link name="t265_pose_frame">
   <inertial>
@@ -191,21 +193,27 @@
   <origin xyz="0 0 0"/>
 </joint>
-<!-- LASER_FRAME TO BASE_LINK -->
+<!-- LASER_LINK TO BASE_LINK -->
 <joint name="base_lidar_fixed" type="fixed">
   <parent link="base_link"/>
+  <child link="laser_link"/>
+  <origin xyz="0 0 0.0415"/>
+</joint>
+<!-- LASER_FRAME TO LASER_LINK -->
+<joint name="laser_frame_fixed" type="fixed">
+  <parent link="laser_link"/>
   <child link="laser_frame"/>
-  <origin xyz="0 0 0.0415"/>
+  <origin xyz="0 0 0.03"/>
 </joint>
 <!-- T265_POSE_FRAME TO BASE_LINK -->
 <joint name="base_t265_fixed" type="fixed">
-  <origin xyz="0.092 0 0.011" rpy="0 0 0" />
   <parent link="base_link" />
   <child link="t265_pose_frame" />
+  <origin xyz="0.092 0 0.011" rpy="0 0 0" />
 </joint>
 <!-- BASE_FOOTPRINT TO BASE_LINK -->
 <joint name="base_link_footprint_fixed" type="fixed">
-  <origin xyz="0 0 -0.063" rpy="0 0 0"/>
   <parent link="base_link"/>
   <child link="base_footprint"/>
+  <origin xyz="0 0 -0.099" rpy="0 0 0"/>
   <axis xyz="0 0 0"/>
 </joint>

Commit message: added joint state publisher to mesh_publisher

File: akros_description/urdf/.ipynb_checkpoints/akros.urdf-checkpoint.xacro (robot description, xacro)
@@ -207,13 +207,13 @@
 <!-- T265_POSE_FRAME TO BASE_LINK -->
 <joint name="base_t265_fixed" type="fixed">
-  <origin xyz="0.092 0 0.011" rpy="0 0 0" />
   <parent link="base_link" />
   <child link="t265_pose_frame" />
+  <origin xyz="0.092 0 0.011" rpy="0 0 0" />
 </joint>
 <!-- BASE_FOOTPRINT TO BASE_LINK -->
 <joint name="base_link_footprint_fixed" type="fixed">
-  <origin xyz="0 0 -0.099" rpy="0 0 0"/>
   <parent link="base_link"/>
   <child link="base_footprint"/>
+  <origin xyz="0 0 -0.099" rpy="0 0 0"/>
   <axis xyz="0 0 0"/>
 </joint>
@@ -228,8 +228,8 @@
   <type>transmission_interface/SimpleTransmission</type>
   <joint name="joint_lf">
-    <hardwareInterface>hardware_interface/EffortJointInterface</hardwareInterface>
+    <hardwareInterface>VelocityJointInterface</hardwareInterface>
   </joint>
   <actuator name="motor_lf">
-    <hardwareInterface>hardware_interface/EffortJointInterface</hardwareInterface>
+    <hardwareInterface>VelocityJointInterface</hardwareInterface>
     <mechanicalReduction>1</mechanicalReduction>
   </actuator>
@@ -245,8 +245,8 @@
   <type>transmission_interface/SimpleTransmission</type>
   <joint name="joint_lb">
-    <hardwareInterface>hardware_interface/EffortJointInterface</hardwareInterface>
+    <hardwareInterface>VelocityJointInterface</hardwareInterface>
   </joint>
   <actuator name="motor_lb">
-    <hardwareInterface>hardware_interface/EffortJointInterface</hardwareInterface>
+    <hardwareInterface>VelocityJointInterface</hardwareInterface>
     <mechanicalReduction>1</mechanicalReduction>
   </actuator>
@@ -262,8 +262,8 @@
   <type>transmission_interface/SimpleTransmission</type>
   <joint name="joint_rf">
-    <hardwareInterface>hardware_interface/EffortJointInterface</hardwareInterface>
+    <hardwareInterface>VelocityJointInterface</hardwareInterface>
   </joint>
   <actuator name="motor_rf">
-    <hardwareInterface>hardware_interface/EffortJointInterface</hardwareInterface>
+    <hardwareInterface>VelocityJointInterface</hardwareInterface>
     <mechanicalReduction>1</mechanicalReduction>
   </actuator>
@@ -279,8 +279,8 @@
   <type>transmission_interface/SimpleTransmission</type>
   <joint name="joint_rb">
-    <hardwareInterface>hardware_interface/EffortJointInterface</hardwareInterface>
+    <hardwareInterface>VelocityJointInterface</hardwareInterface>
   </joint>
   <actuator name="motor_rb">
-    <hardwareInterface>hardware_interface/EffortJointInterface</hardwareInterface>
+    <hardwareInterface>VelocityJointInterface</hardwareInterface>
     <mechanicalReduction>1</mechanicalReduction>
   </actuator>
@@ -352,6 +352,6 @@
   </plugin>
 </gazebo>
-<!--<gazebo>
+<!-- gazebo>
   <plugin name="control" filename="libgazebo_ros_control.so"/>
-</gazebo>-->
+</gazebo> -->
 </robot>

File: akros_description/urdf/akros.urdf.xacro (robot description, xacro)
@@ -228,8 +228,8 @@
   <type>transmission_interface/SimpleTransmission</type>
   <joint name="joint_lf">
-    <hardwareInterface>hardware_interface/EffortJointInterface</hardwareInterface>
+    <hardwareInterface>VelocityJointInterface</hardwareInterface>
   </joint>
   <actuator name="motor_lf">
-    <hardwareInterface>hardware_interface/EffortJointInterface</hardwareInterface>
+    <hardwareInterface>VelocityJointInterface</hardwareInterface>
     <mechanicalReduction>1</mechanicalReduction>
   </actuator>
@@ -245,8 +245,8 @@
   <type>transmission_interface/SimpleTransmission</type>
   <joint name="joint_lb">
-    <hardwareInterface>hardware_interface/EffortJointInterface</hardwareInterface>
+    <hardwareInterface>VelocityJointInterface</hardwareInterface>
   </joint>
   <actuator name="motor_lb">
-    <hardwareInterface>hardware_interface/EffortJointInterface</hardwareInterface>
+    <hardwareInterface>VelocityJointInterface</hardwareInterface>
     <mechanicalReduction>1</mechanicalReduction>
   </actuator>
@@ -262,8 +262,8 @@
   <type>transmission_interface/SimpleTransmission</type>
   <joint name="joint_rf">
-    <hardwareInterface>hardware_interface/EffortJointInterface</hardwareInterface>
+    <hardwareInterface>VelocityJointInterface</hardwareInterface>
   </joint>
   <actuator name="motor_rf">
-    <hardwareInterface>hardware_interface/EffortJointInterface</hardwareInterface>
+    <hardwareInterface>VelocityJointInterface</hardwareInterface>
     <mechanicalReduction>1</mechanicalReduction>
   </actuator>
@@ -279,8 +279,8 @@
   <type>transmission_interface/SimpleTransmission</type>
   <joint name="joint_rb">
-    <hardwareInterface>hardware_interface/EffortJointInterface</hardwareInterface>
+    <hardwareInterface>VelocityJointInterface</hardwareInterface>
   </joint>
   <actuator name="motor_rb">
-    <hardwareInterface>hardware_interface/EffortJointInterface</hardwareInterface>
+    <hardwareInterface>VelocityJointInterface</hardwareInterface>
     <mechanicalReduction>1</mechanicalReduction>
   </actuator>
@@ -352,6 +352,6 @@
   </plugin>
 </gazebo>
-<!--<gazebo>
+<!-- gazebo>
   <plugin name="control" filename="libgazebo_ros_control.so"/>
-</gazebo>-->
+</gazebo> -->
 </robot>
